Commit message: Added inertia macros

File: src/robot_description/resource/robot.urdf.xacro (robot description, xacro)
@@ -1,7 +1,9 @@
 <?xml version="1.0"?>
 <robot name="robot" xmlns:xacro="http://ros.org/wiki/xacro">
-    <link name="base_footprint">
+    <xacro:include filename="$(find robot_description)/resource/macros.urdf.xacro" />
+    <link name="base_link">
+        <xacro:box_inertia m="0" w="0" d="0" h="0"/>
     </link>
-    <link name="base_link">
+    <link name="body_link">
         <visual>
             <geometry>
@@ -14,8 +16,9 @@
             </geometry>
         </collision>
+        <xacro:box_inertia m="1" w="1" d="1" h="1"/>
     </link>
     <joint name="base_joint" type="fixed">
         <parent link="base_link" />
-        <child link="base_footprint" />
+        <child link="body_link" />
         <origin xyz="0.0 0.0 1.0" rpy="0 0 0" />
     </joint>

Commit message: Driving platform

File: src/robot_description/resource/robot.urdf.xacro (robot description, xacro)
@@ -1,25 +1,109 @@
 <?xml version="1.0"?>
-<robot name="robot" xmlns:xacro="http://ros.org/wiki/xacro">
+<robot name="my_robot" xmlns:xacro="http://ros.org/wiki/xacro">
     <xacro:include filename="$(find robot_description)/resource/macros.urdf.xacro" />
     <link name="base_link">
-        <xacro:box_inertia m="0" w="0" d="0" h="0"/>
+        <!-- <xacro:box_inertia m="0" w="0" d="0" h="0"/> -->
     </link>
+    <xacro:property name="base_width" value="0.31" />
+    <xacro:property name="base_length" value="0.42" />
+    <xacro:property name="base_height" value="0.18" />
+    <xacro:property name="base_mass" value="1.0" />
+    <xacro:property name="wheel_radius" value="0.10" />
+    <xacro:property name="wheel_width" value="0.04" />
+    <xacro:property name="wheel_ygap" value="0.025" />
+    <xacro:property name="wheel_zoff" value="0.05" />
+    <xacro:property name="wheel_xoff" value="0.12" />
+    <xacro:property name="wheel_mass" value="0.1" />
+    <xacro:property name="caster_xoff" value="0.14" />
     <link name="body_link">
         <visual>
             <geometry>
-                <box size="1.0 1.0 1.0" />
+                <box size="${base_length} ${base_width}  ${base_height}" />
             </geometry>
         </visual>
         <collision>
             <geometry>
-                <box size="1.0 1.0 1.0" />
+                <box size="${base_length} ${base_width} ${base_height}" />
             </geometry>
         </collision>
-        <xacro:box_inertia m="1" w="1" d="1" h="1"/>
+        <xacro:box_inertia m="${base_mass}" w="${base_width}" d="${base_length}" h="${base_height}" />
     </link>
     <joint name="base_joint" type="fixed">
         <parent link="base_link" />
         <child link="body_link" />
-        <origin xyz="0.0 0.0 1.0" rpy="0 0 0" />
+        <origin xyz="0.0 0.0  ${-(wheel_radius+wheel_zoff)}" rpy="0 0 0" />
     </joint>
+    <!-- Wheels -->
+    <xacro:macro name="wheel" params="prefix x_reflect y_reflect">
+        <link name="${prefix}_link">
+            <visual>
+                <origin xyz="0 0 0" rpy="${pi/2} 0 0" />
+                <geometry>
+                    <cylinder radius="${wheel_radius}" length="${wheel_width}" />
+                </geometry>
+                <material name="Gray">
+                    <color rgba="0.5 0.5 0.5 1.0" />
+                </material>
+            </visual>
+            <collision>
+                <origin xyz="0 0 0" rpy="${pi/2} 0 0" />
+                <geometry>
+                    <cylinder radius="${wheel_radius}" length="${wheel_width}" />
+                </geometry>
+            </collision>
+            <xacro:cylinder_inertia m="${wheel_mass}" r="${wheel_radius}" h="${wheel_width}" />
+        </link>
+        <joint name="${prefix}_joint" type="continuous">
+            <parent link="body_link" />
+            <child link="${prefix}_link" />
+            <origin xyz="${x_reflect*wheel_xoff} ${y_reflect*(base_width/2+wheel_ygap)} ${-wheel_zoff}" rpy="0 0 0" />
+            <axis xyz="0 1 0" />
+        </joint>
+    </xacro:macro>
+    <xacro:wheel prefix="drivewhl_l" x_reflect="-1" y_reflect="1" />
+    <xacro:wheel prefix="drivewhl_r" x_reflect="-1" y_reflect="-1" />
+    <!-- Caster Wheel -->
+    <link name="front_caster">
+        <visual>
+            <geometry>
+                <sphere radius="${(wheel_radius+wheel_zoff-(base_height/2))}" />
+            </geometry>
+            <material name="Cyan">
+                <color rgba="0 1.0 1.0 1.0" />
+            </material>
+        </visual>
+        <collision>
+            <geometry>
+                <sphere radius="${(wheel_radius+wheel_zoff-(base_height/2))}" />
+            </geometry>
+        </collision>
+    </link>
+    <joint name="caster_joint" type="fixed">
+        <parent link="body_link" />
+        <child link="front_caster" />
+        <origin xyz="${caster_xoff} 0.0 ${-(base_height/2)}" rpy="0 0 0" />
+    </joint>
+    <gazebo reference="front_caster">
+        <mu>0.001</mu>
+        <mu2>0.001</mu2>
+    </gazebo>
+    <gazebo>
+        <plugin name='diff_drive' filename='libgazebo_ros_diff_drive.so'>
+            <!-- wheels -->
+            <left_joint>drivewhl_l_joint</left_joint>
+            <right_joint>drivewhl_r_joint</right_joint>
+            <!-- kinematics -->
+            <wheel_separation>0.4</wheel_separation>
+            <wheel_diameter>0.2</wheel_diameter>
+            <!-- limits -->
+            <max_wheel_torque>20</max_wheel_torque>
+            <max_wheel_acceleration>1.0</max_wheel_acceleration>
+            <!-- output -->
+            <publish_odom>true</publish_odom>
+            <publish_odom_tf>false</publish_odom_tf>
+            <publish_wheel_tf>true</publish_wheel_tf>
+            <odometry_frame>odom</odometry_frame>
+            <robot_base_frame>body_link</robot_base_frame>
+        </plugin>
+    </gazebo>
 </robot>

Commit message: Added lidar

File: src/robot_description/resource/robot.urdf.xacro (robot description, xacro)
@@ -2,7 +2,5 @@
 <robot name="my_robot" xmlns:xacro="http://ros.org/wiki/xacro">
     <xacro:include filename="$(find robot_description)/resource/macros.urdf.xacro" />
-    <link name="base_link">
-        <!-- <xacro:box_inertia m="0" w="0" d="0" h="0"/> -->
-    </link>
+    <link name="base_footprint"/>
     <xacro:property name="base_width" value="0.31" />
     <xacro:property name="base_length" value="0.42" />
@@ -16,5 +14,5 @@
     <xacro:property name="wheel_mass" value="0.1" />
     <xacro:property name="caster_xoff" value="0.14" />
-    <link name="body_link">
+    <link name="base_link">
         <visual>
             <geometry>
@@ -30,7 +28,7 @@
     </link>
     <joint name="base_joint" type="fixed">
-        <parent link="base_link" />
-        <child link="body_link" />
-        <origin xyz="0.0 0.0  ${-(wheel_radius+wheel_zoff)}" rpy="0 0 0" />
+        <parent link="base_footprint" />
+        <child link="base_link" />
+        <origin xyz="0.0 0.0  ${(wheel_radius+wheel_zoff)}" rpy="0 0 0" />
     </joint>
     <!-- Wheels -->
@@ -55,5 +53,5 @@
         </link>
         <joint name="${prefix}_joint" type="continuous">
-            <parent link="body_link" />
+            <parent link="base_link" />
             <child link="${prefix}_link" />
             <origin xyz="${x_reflect*wheel_xoff} ${y_reflect*(base_width/2+wheel_ygap)} ${-wheel_zoff}" rpy="0 0 0" />
@@ -80,11 +78,31 @@
     </link>
     <joint name="caster_joint" type="fixed">
-        <parent link="body_link" />
+        <parent link="base_link" />
         <child link="front_caster" />
         <origin xyz="${caster_xoff} 0.0 ${-(base_height/2)}" rpy="0 0 0" />
     </joint>
+    <link name="lidar_link">
+        <collision>
+            <origin xyz="0 0 0" rpy="0 0 0" />
+            <geometry>
+                <cylinder radius="0.0508" length="0.055" />
+            </geometry>
+        </collision>
+        <visual>
+            <origin xyz="0 0 0" rpy="0 0 0" />
+            <geometry>
+                <cylinder radius="0.0508" length="0.055" />
+            </geometry>
+        </visual>
+        <xacro:cylinder_inertia m="0.125" r="0.0508" h="0.055" />
+    </link>
+    <joint name="lidar_joint" type="fixed">
+        <parent link="base_link" />
+        <child link="lidar_link" />
+        <origin xyz="0 0 0.12" rpy="0 0 0" />
+    </joint>
     <gazebo reference="front_caster">
-        <mu>0.001</mu>
-        <mu2>0.001</mu2>
+        <mu>0.0</mu>
+        <mu2>0.0</mu2>
     </gazebo>
     <gazebo>
@@ -101,9 +119,43 @@
             <!-- output -->
             <publish_odom>true</publish_odom>
-            <publish_odom_tf>false</publish_odom_tf>
+            <publish_odom_tf>true</publish_odom_tf>
             <publish_wheel_tf>true</publish_wheel_tf>
             <odometry_frame>odom</odometry_frame>
-            <robot_base_frame>body_link</robot_base_frame>
+            <robot_base_frame>base_footprint</robot_base_frame>
         </plugin>
     </gazebo>
+    <gazebo reference="lidar_link">
+        <sensor name="lidar" type="ray">
+            <always_on>true</always_on>
+            <visualize>true</visualize>
+            <update_rate>5</update_rate>
+            <ray>
+                <scan>
+                    <horizontal>
+                        <samples>360</samples>
+                        <resolution>1.000000</resolution>
+                        <min_angle>0.000000</min_angle>
+                        <max_angle>6.280000</max_angle>
+                    </horizontal>
+                </scan>
+                <range>
+                    <min>0.120000</min>
+                    <max>3.5</max>
+                    <resolution>0.015000</resolution>
+                </range>
+                <noise>
+                    <type>gaussian</type>
+                    <mean>0.0</mean>
+                    <stddev>0.01</stddev>
+                </noise>
+            </ray>
+            <plugin name="scan" filename="libgazebo_ros_ray_sensor.so">
+                <ros>
+                    <remapping>~/out:=scan</remapping>
+                </ros>
+                <output_type>sensor_msgs/LaserScan</output_type>
+                <frame_name>lidar_link</frame_name>
+            </plugin>
+        </sensor>
+    </gazebo>
 </robot>

Commit message: dziala

File: src/robot_description/resource/robot.urdf.xacro (robot description, xacro)
@@ -6,5 +6,5 @@
     <xacro:property name="base_length" value="0.42" />
     <xacro:property name="base_height" value="0.18" />
-    <xacro:property name="base_mass" value="1.0" />
+    <xacro:property name="base_mass" value="5.0" />
     <xacro:property name="wheel_radius" value="0.10" />
     <xacro:property name="wheel_width" value="0.04" />
@@ -58,4 +58,9 @@
             <axis xyz="0 1 0" />
         </joint>
+        <gazebo reference="${prefix}_link">
+            <mu1 value="10.0" />
+            <mu2 value="10.0" />
+        <material>Gazebo/Black</material>
+    </gazebo>
     </xacro:macro>
     <xacro:wheel prefix="drivewhl_l" x_reflect="-1" y_reflect="1" />
@@ -103,6 +108,7 @@
     </joint>
     <gazebo reference="front_caster">
-        <mu>0.0</mu>
-        <mu2>0.0</mu2>
+        <mu1 value="0.00000001" />
+        <mu2 value="0.00000001" />
+        <material>Gazebo/Black</material>
     </gazebo>
     <gazebo>
@@ -115,6 +121,6 @@
             <wheel_diameter>0.2</wheel_diameter>
             <!-- limits -->
-            <max_wheel_torque>20</max_wheel_torque>
-            <max_wheel_acceleration>1.0</max_wheel_acceleration>
+            <max_wheel_torque>40</max_wheel_torque>
+            <max_wheel_acceleration>2.0</max_wheel_acceleration>
             <!-- output -->
             <publish_odom>true</publish_odom>

Commit message: start

File: src/robot_description/resource/robot.urdf.xacro (robot description, xacro)
@@ -3,165 +3,20 @@
     <xacro:include filename="$(find robot_description)/resource/macros.urdf.xacro" />
     <link name="base_footprint"/>
-    <xacro:property name="base_width" value="0.31" />
-    <xacro:property name="base_length" value="0.42" />
-    <xacro:property name="base_height" value="0.18" />
-    <xacro:property name="base_mass" value="5.0" />
-    <xacro:property name="wheel_radius" value="0.10" />
-    <xacro:property name="wheel_width" value="0.04" />
-    <xacro:property name="wheel_ygap" value="0.025" />
-    <xacro:property name="wheel_zoff" value="0.05" />
-    <xacro:property name="wheel_xoff" value="0.12" />
-    <xacro:property name="wheel_mass" value="0.1" />
-    <xacro:property name="caster_xoff" value="0.14" />
     <link name="base_link">
         <visual>
             <geometry>
-                <box size="${base_length} ${base_width}  ${base_height}" />
+                <box size="1.0 1.0 1.0" />
             </geometry>
         </visual>
         <collision>
             <geometry>
-                <box size="${base_length} ${base_width} ${base_height}" />
+                <box size="1.0 1.0 1.0" />
             </geometry>
         </collision>
-        <xacro:box_inertia m="${base_mass}" w="${base_width}" d="${base_length}" h="${base_height}" />
     </link>
     <joint name="base_joint" type="fixed">
         <parent link="base_footprint" />
         <child link="base_link" />
-        <origin xyz="0.0 0.0  ${(wheel_radius+wheel_zoff)}" rpy="0 0 0" />
+        <origin xyz="0.0 0.0  1.0" rpy="0 0 0" />
     </joint>
-    <!-- Wheels -->
-    <xacro:macro name="wheel" params="prefix x_reflect y_reflect">
-        <link name="${prefix}_link">
-            <visual>
-                <origin xyz="0 0 0" rpy="${pi/2} 0 0" />
-                <geometry>
-                    <cylinder radius="${wheel_radius}" length="${wheel_width}" />
-                </geometry>
-                <material name="Gray">
-                    <color rgba="0.5 0.5 0.5 1.0" />
-                </material>
-            </visual>
-            <collision>
-                <origin xyz="0 0 0" rpy="${pi/2} 0 0" />
-                <geometry>
-                    <cylinder radius="${wheel_radius}" length="${wheel_width}" />
-                </geometry>
-            </collision>
-            <xacro:cylinder_inertia m="${wheel_mass}" r="${wheel_radius}" h="${wheel_width}" />
-        </link>
-        <joint name="${prefix}_joint" type="continuous">
-            <parent link="base_link" />
-            <child link="${prefix}_link" />
-            <origin xyz="${x_reflect*wheel_xoff} ${y_reflect*(base_width/2+wheel_ygap)} ${-wheel_zoff}" rpy="0 0 0" />
-            <axis xyz="0 1 0" />
-        </joint>
-        <gazebo reference="${prefix}_link">
-            <mu1 value="10.0" />
-            <mu2 value="10.0" />
-        <material>Gazebo/Black</material>
-    </gazebo>
-    </xacro:macro>
-    <xacro:wheel prefix="drivewhl_l" x_reflect="-1" y_reflect="1" />
-    <xacro:wheel prefix="drivewhl_r" x_reflect="-1" y_reflect="-1" />
-    <!-- Caster Wheel -->
-    <link name="front_caster">
-        <visual>
-            <geometry>
-                <sphere radius="${(wheel_radius+wheel_zoff-(base_height/2))}" />
-            </geometry>
-            <material name="Cyan">
-                <color rgba="0 1.0 1.0 1.0" />
-            </material>
-        </visual>
-        <collision>
-            <geometry>
-                <sphere radius="${(wheel_radius+wheel_zoff-(base_height/2))}" />
-            </geometry>
-        </collision>
-    </link>
-    <joint name="caster_joint" type="fixed">
-        <parent link="base_link" />
-        <child link="front_caster" />
-        <origin xyz="${caster_xoff} 0.0 ${-(base_height/2)}" rpy="0 0 0" />
-    </joint>
-    <link name="lidar_link">
-        <collision>
-            <origin xyz="0 0 0" rpy="0 0 0" />
-            <geometry>
-                <cylinder radius="0.0508" length="0.055" />
-            </geometry>
-        </collision>
-        <visual>
-            <origin xyz="0 0 0" rpy="0 0 0" />
-            <geometry>
-                <cylinder radius="0.0508" length="0.055" />
-            </geometry>
-        </visual>
-        <xacro:cylinder_inertia m="0.125" r="0.0508" h="0.055" />
-    </link>
-    <joint name="lidar_joint" type="fixed">
-        <parent link="base_link" />
-        <child link="lidar_link" />
-        <origin xyz="0 0 0.12" rpy="0 0 0" />
-    </joint>
-    <gazebo reference="front_caster">
-        <mu1 value="0.00000001" />
-        <mu2 value="0.00000001" />
-        <material>Gazebo/Black</material>
-    </gazebo>
-    <gazebo>
-        <plugin name='diff_drive' filename='libgazebo_ros_diff_drive.so'>
-            <!-- wheels -->
-            <left_joint>drivewhl_l_joint</left_joint>
-            <right_joint>drivewhl_r_joint</right_joint>
-            <!-- kinematics -->
-            <wheel_separation>0.4</wheel_separation>
-            <wheel_diameter>0.2</wheel_diameter>
-            <!-- limits -->
-            <max_wheel_torque>40</max_wheel_torque>
-            <max_wheel_acceleration>2.0</max_wheel_acceleration>
-            <!-- output -->
-            <publish_odom>true</publish_odom>
-            <publish_odom_tf>true</publish_odom_tf>
-            <publish_wheel_tf>true</publish_wheel_tf>
-            <odometry_frame>odom</odometry_frame>
-            <robot_base_frame>base_footprint</robot_base_frame>
-        </plugin>
-    </gazebo>
-    <gazebo reference="lidar_link">
-        <sensor name="lidar" type="ray">
-            <always_on>true</always_on>
-            <visualize>true</visualize>
-            <update_rate>5</update_rate>
-            <ray>
-                <scan>
-                    <horizontal>
-                        <samples>360</samples>
-                        <resolution>1.000000</resolution>
-                        <min_angle>0.000000</min_angle>
-                        <max_angle>6.280000</max_angle>
-                    </horizontal>
-                </scan>
-                <range>
-                    <min>0.120000</min>
-                    <max>3.5</max>
-                    <resolution>0.015000</resolution>
-                </range>
-                <noise>
-                    <type>gaussian</type>
-                    <mean>0.0</mean>
-                    <stddev>0.01</stddev>
-                </noise>
-            </ray>
-            <plugin name="scan" filename="libgazebo_ros_ray_sensor.so">
-                <ros>
-                    <remapping>~/out:=scan</remapping>
-                </ros>
-                <output_type>sensor_msgs/LaserScan</output_type>
-                <frame_name>lidar_link</frame_name>
-            </plugin>
-        </sensor>
-    </gazebo>
 </robot>
