Commit message: reverted changes

File: src/robot_description/resource/robot.urdf.xacro (robot description, xacro)
@@ -2,27 +2,14 @@
 <robot name="my_robot" xmlns:xacro="http://ros.org/wiki/xacro">
     <xacro:include filename="$(find robot_description)/resource/macros.urdf.xacro" />
-    <xacro:property name="base_width" value="0.31" />
-    <xacro:property name="base_length" value="0.42" />
-    <xacro:property name="base_height" value="0.18" />
-    <xacro:property name="base_mass" value="1.0" />
-    <xacro:property name="wheel_radius" value="0.10" />
-    <xacro:property name="wheel_width" value="0.04" />
-    <xacro:property name="wheel_ygap" value="0.025" />
-    <xacro:property name="wheel_zoff" value="0.05" />
-    <xacro:property name="wheel_xoff" value="0.12" />
-    <xacro:property name="wheel_mass" value="0.5" />
-    <xacro:property name="caster_xoff" value="0.15" />
-    <xacro:property name="caster_mass" value="0.10" />
-    <link name="base_footprint" />
+    <link name="base_footprint"/>
     <link name="base_link">
-        <xacro:box_inertia m="${base_mass}" w="${base_width}" d="${base_length}" h="${base_height}" />
         <visual>
             <geometry>
-                <box size="${base_length} ${base_width} ${base_height}" />
+                <box size="1.0 1.0 1.0" />
             </geometry>
         </visual>
         <collision>
             <geometry>
-                <box size="${base_length} ${base_width} ${base_height}" />
+                <box size="1.0 1.0 1.0" />
             </geometry>
         </collision>
@@ -31,133 +18,5 @@
         <parent link="base_footprint" />
         <child link="base_link" />
-        <origin xyz="0.0 0.0  ${wheel_radius + base_height/2}" rpy="0 0 0" />
+        <origin xyz="0.0 0.0  1.0" rpy="0 0 0" />
     </joint>
-    <xacro:macro name="wheel" params="prefix x_reflect y_reflect">
-        <link name="${prefix}_link">
-            <visual>
-                <origin xyz="0 0 0" rpy="${pi/2} 0 0" />
-                <geometry>
-                    <cylinder radius="${wheel_radius}" length="${wheel_width}" />
-                </geometry>
-                <material name="Gray">
-                    <color rgba="0.5 0.5 0.5 1.0" />
-                </material>
-            </visual>
-            <collision>
-                <origin xyz="0 0 0" rpy="${pi/2} 0 0" />
-                <geometry>
-                    <cylinder radius="${wheel_radius}" length="${wheel_width}" />
-                </geometry>
-            </collision>
-            <xacro:cylinder_inertia m="${wheel_mass}" r="${wheel_radius}" h="${wheel_width}" />
-        </link>
-        <joint name="${prefix}_joint" type="continuous">
-            <parent link="base_link" />
-            <child link="${prefix}_link" />
-            <origin
-                xyz="${x_reflect*wheel_xoff} ${y_reflect*(base_width/2+wheel_ygap)} ${-wheel_zoff}"
-                rpy="0 0 0" />
-            <axis xyz="0 1 0" />
-        </joint>
-    </xacro:macro>
-    <xacro:wheel prefix="drivewhl_l" x_reflect="-1" y_reflect="1" />
-    <xacro:wheel prefix="drivewhl_r" x_reflect="-1" y_reflect="-1" />
-    <link name="front_caster">
-        <visual>
-            <geometry>
-                <sphere radius="${(wheel_radius+wheel_zoff-(base_height/2))}" />
-            </geometry>
-            <material name="Cyan">
-                <color rgba="0 1.0 1.0 1.0" />
-            </material>
-        </visual>
-        <collision>
-            <geometry>
-                <sphere radius="${(wheel_radius+wheel_zoff-(base_height/2))}" />
-            </geometry>
-        </collision>
-        <xacro:sphere_inertia m="${caster_mass}" r="${(wheel_radius+wheel_zoff-(base_height/2))}" />
-    </link>
-    <joint name="caster_joint" type="fixed">
-        <parent link="base_link" />
-        <child link="front_caster" />
-        <origin xyz="${caster_xoff} 0.0 ${-(base_height/2)}" rpy="0 0 0" />
-    </joint>
-    <gazebo reference="front_caster">
-        <mu>0.001</mu>
-        <mu2>0.001</mu2>
-    </gazebo>
-    <gazebo>
-        <plugin name='diff_drive' filename='libgazebo_ros_diff_drive.so'>
-            <!-- wheels -->
-            <left_joint>drivewhl_l_joint</left_joint>
-            <right_joint>drivewhl_r_joint</right_joint>
-            <!-- kinematics -->
-            <wheel_separation>0.4</wheel_separation>
-            <wheel_diameter>0.2</wheel_diameter>
-            <!-- limits -->
-            <max_wheel_torque>20</max_wheel_torque>
-            <max_wheel_acceleration>1.0</max_wheel_acceleration>
-            <!-- output -->
-            <publish_odom>true</publish_odom>
-            <publish_odom_tf>true</publish_odom_tf>
-            <publish_wheel_tf>true</publish_wheel_tf>
-            <odometry_frame>odom</odometry_frame>
-            <robot_base_frame>base_footprint</robot_base_frame>
-        </plugin>
-    </gazebo>
-    <link name="lidar_link">
-        <xacro:cylinder_inertia m="0.1" r="0.0508" h="0.055" />
-        <collision>
-            <origin xyz="0 0 0" rpy="0 0 0" />
-            <geometry>
-                <cylinder radius="0.0508" length="0.055" />
-            </geometry>
-        </collision>
-        <visual>
-            <origin xyz="0 0 0" rpy="0 0 0" />
-            <geometry>
-                <cylinder radius="0.0508" length="0.055" />
-            </geometry>
-        </visual>
-    </link>
-    <joint name="lidar_joint" type="fixed">
-        <parent link="base_link" />
-        <child link="lidar_link" />
-        <origin xyz="0 0 ${base_height/2 + 0.0225}" rpy="0 0 0" />
-    </joint>
-    <gazebo reference="lidar_link">
-        <sensor name="lidar" type="ray">
-            <always_on>true</always_on>
-            <visualize>true</visualize>
-            <update_rate>5</update_rate>
-            <ray>
-                <scan>
-                    <horizontal>
-                        <samples>360</samples>
-                        <resolution>1.000000</resolution>
-                        <min_angle>0.000000</min_angle>
-                        <max_angle>6.280000</max_angle>
-                    </horizontal>
-                </scan>
-                <range>
-                    <min>0.120000</min>
-                    <max>3.5</max>
-                    <resolution>0.015000</resolution>
-                </range>
-                <noise>
-                    <type>gaussian</type>
-                    <mean>0.0</mean>
-                    <stddev>0.01</stddev>
-                </noise>
-            </ray>
-            <plugin name="scan" filename="libgazebo_ros_ray_sensor.so">
-                <ros>
-                    <remapping>~/out:=scan</remapping>
-                </ros>
-                <output_type>sensor_msgs/LaserScan</output_type>
-                <frame_name>lidar_link</frame_name>
-            </plugin>
-        </sensor>
-    </gazebo>
 </robot>
